Commit message: Update quadrotor_with_cam.urdf.xacro
Signed-off-by: TexnoMann <ElectroDans@yandex.ru>

File: hector_quadrotor_description/urdf/quadrotor_with_cam.urdf.xacro (robot description, xacro)
@@ -8,6 +8,10 @@
     <!-- Forward facing camera -->
     <xacro:include filename="$(find hector_sensors_description)/urdf/generic_camera.urdf.xacro" />
-    <xacro:generic_camera name="front_cam" parent="base_link" ros_topic="camera/image" cam_info_topic="camera/camera_info" update_rate="10" res_x="320" res_y="240" image_format="R8G8B8" hfov="90">
-      <origin xyz="0.05 0.0 -0.06" rpy="0 0 0"/>
+    <xacro:generic_camera name="cam_1" parent="base_link" ros_topic="camera/image" cam_info_topic="camera/camera_info" update_rate="30" res_x="320" res_y="240" image_format="R8G8B8" hfov="90">
+      <origin xyz="0.0 0.0 -0.1" rpy="0 1.5707963267948966 0"/>
+    </xacro:generic_camera>
+    <xacro:include filename="$(find hector_sensors_description)/urdf/generic_camera.urdf.xacro" />
+    <xacro:generic_camera name="cam_2" parent="base_link" ros_topic="camera/image" cam_info_topic="camera/camera_info" update_rate="30" res_x="320" res_y="240" image_format="R8G8B8" hfov="90">
+      <origin xyz="0.0 -0.0 -0.2" rpy="0 0 0"/>
     </xacro:generic_camera>
 </robot>
